Commit message: Robot model: 2 mm gap between adjacent parts (user request, reviewed in RViz)
Every joint origin moves 2 mm along its axis toward the child, so the flat faces at all six
joints are 2.00 mm apart instead of touching (measured on the meshes); the parent's 9 mm
boss now sits 7 mm deep in the child's bore. Meshes unchanged.

- urdf/6dof.urdf, urdf/6dof.xacro, mujoco/6dof_mj.urdf, 6dof.xml, 6dof_control.xml
- regenerated: urdf/6dof_gripper.{urdf,xacro}, models/generated/pinch_scene.xml
- ready pose kept in joint space; its TCP is now +2 mm x, +2 mm y (no contacts, floor
  clearance 43.6 mm, self clearance 11.7 mm)
- model hash reference updated; target-grid scan 78/78 still passes all 12 checks

Co-Authored-By: Claude Opus 5.5 <noreply@anthropic.com>

File: 6dof_description/mujoco/6dof_mj.urdf (robot description, URDF)
Before this commit: robot 6dof, 7 links, 6 joints
Joints:
- joint Revolute_1: origin xyz=0.0 0.002984 0.041554 rpy=0 0 0 -> xyz=0.0 0.002984 0.043554 rpy=0 0 0
- joint Revolute_2: origin xyz=0.04 0.0 0.0505 rpy=0 0 0 -> xyz=0.042 0.0 0.0505 rpy=0 0 0
- joint Revolute_3: origin xyz=0.0 0.0 0.2 rpy=0 0 0 -> xyz=-0.002 0.0 0.2 rpy=0 0 0
- joint Revolute_4: origin xyz=0.0 0.0 0.2 rpy=0 0 0 -> xyz=0.002 0.0 0.2 rpy=0 0 0
- joint Revolute_5: origin xyz=0.0505 0.0 0.04 rpy=0 0 0 -> xyz=0.0505 0.0 0.042 rpy=0 0 0
- joint Revolute_6: origin xyz=-0.04 0.0 0.0505 rpy=0 0 0 -> xyz=-0.042 0.0 0.0505 rpy=0 0 0

File: 6dof_description/urdf/6dof.urdf (robot description, URDF)
Before this commit: robot 6dof, 7 links, 6 joints
Joints:
- joint Revolute_1: origin xyz=0.0 0.002984 0.041554 rpy=0 0 0 -> xyz=0.0 0.002984 0.043554 rpy=0 0 0
- joint Revolute_2: origin xyz=0.04 0.0 0.0505 rpy=0 0 0 -> xyz=0.042 0.0 0.0505 rpy=0 0 0
- joint Revolute_3: origin xyz=0.0 0.0 0.2 rpy=0 0 0 -> xyz=-0.002 0.0 0.2 rpy=0 0 0
- joint Revolute_4: origin xyz=0.0 0.0 0.2 rpy=0 0 0 -> xyz=0.002 0.0 0.2 rpy=0 0 0
- joint Revolute_5: origin xyz=0.0505 0.0 0.04 rpy=0 0 0 -> xyz=0.0505 0.0 0.042 rpy=0 0 0
- joint Revolute_6: origin xyz=-0.04 0.0 0.0505 rpy=0 0 0 -> xyz=-0.042 0.0 0.0505 rpy=0 0 0

File: 6dof_description/urdf/6dof.xacro (robot description, xacro)
@@ -143,5 +143,5 @@
 </link>
 <joint name="Revolute_1" type="revolute">
-  <origin xyz="0.0 0.002984 0.041554" rpy="0 0 0"/>
+  <origin xyz="0.0 0.002984 0.043554" rpy="0 0 0"/>
   <parent link="base_link"/>
   <child link="r_a_1"/>
@@ -150,5 +150,5 @@
 </joint>
 <joint name="Revolute_2" type="revolute">
-  <origin xyz="0.04 0.0 0.0505" rpy="0 0 0"/>
+  <origin xyz="0.042 0.0 0.0505" rpy="0 0 0"/>
   <parent link="r_a_1"/>
   <child link="link_1"/>
@@ -157,5 +157,5 @@
 </joint>
 <joint name="Revolute_3" type="revolute">
-  <origin xyz="0.0 0.0 0.2" rpy="0 0 0"/>
+  <origin xyz="-0.002 0.0 0.2" rpy="0 0 0"/>
   <parent link="link_1"/>
   <child link="link__1__1"/>
@@ -164,5 +164,5 @@
 </joint>
 <joint name="Revolute_4" type="revolute">
-  <origin xyz="0.0 0.0 0.2" rpy="0 0 0"/>
+  <origin xyz="0.002 0.0 0.2" rpy="0 0 0"/>
   <parent link="link__1__1"/>
   <child link="r_a__1__1"/>
@@ -171,5 +171,5 @@
 </joint>
 <joint name="Revolute_5" type="revolute">
-  <origin xyz="0.0505 0.0 0.04" rpy="0 0 0"/>
+  <origin xyz="0.0505 0.0 0.042" rpy="0 0 0"/>
   <parent link="r_a__1__1"/>
   <child link="r_a__2__1"/>
@@ -178,5 +178,5 @@
 </joint>
 <joint name="Revolute_6" type="revolute">
-  <origin xyz="-0.04 0.0 0.0505" rpy="0 0 0"/>
+  <origin xyz="-0.042 0.0 0.0505" rpy="0 0 0"/>
   <parent link="r_a__2__1"/>
   <child link="housing_1"/>

File: 6dof_description/urdf/6dof_gripper.urdf (robot description, URDF)
Before this commit: robot 6dof_gripper, 7 links, 6 joints
Joints:
- joint Revolute_1: origin xyz=0.0 0.002984 0.041554 rpy=0 0 0 -> xyz=0.0 0.002984 0.043554 rpy=0 0 0
- joint Revolute_2: origin xyz=0.04 0.0 0.0505 rpy=0 0 0 -> xyz=0.042 0.0 0.0505 rpy=0 0 0
- joint Revolute_3: origin xyz=0.0 0.0 0.2 rpy=0 0 0 -> xyz=-0.002 0.0 0.2 rpy=0 0 0
- joint Revolute_4: origin xyz=0.0 0.0 0.2 rpy=0 0 0 -> xyz=0.002 0.0 0.2 rpy=0 0 0
- joint Revolute_5: origin xyz=0.0505 0.0 0.04 rpy=0 0 0 -> xyz=0.0505 0.0 0.042 rpy=0 0 0
- joint Revolute_6: origin xyz=-0.04 0.0 0.0505 rpy=0 0 0 -> xyz=-0.042 0.0 0.0505 rpy=0 0 0

File: 6dof_description/urdf/6dof_gripper.xacro (robot description, xacro)
@@ -144,5 +144,5 @@
 </link>
 <joint name="Revolute_1" type="revolute">
-  <origin xyz="0.0 0.002984 0.041554" rpy="0 0 0"/>
+  <origin xyz="0.0 0.002984 0.043554" rpy="0 0 0"/>
   <parent link="base_link"/>
   <child link="r_a_1"/>
@@ -151,5 +151,5 @@
 </joint>
 <joint name="Revolute_2" type="revolute">
-  <origin xyz="0.04 0.0 0.0505" rpy="0 0 0"/>
+  <origin xyz="0.042 0.0 0.0505" rpy="0 0 0"/>
   <parent link="r_a_1"/>
   <child link="link_1"/>
@@ -158,5 +158,5 @@
 </joint>
 <joint name="Revolute_3" type="revolute">
-  <origin xyz="0.0 0.0 0.2" rpy="0 0 0"/>
+  <origin xyz="-0.002 0.0 0.2" rpy="0 0 0"/>
   <parent link="link_1"/>
   <child link="link__1__1"/>
@@ -165,5 +165,5 @@
 </joint>
 <joint name="Revolute_4" type="revolute">
-  <origin xyz="0.0 0.0 0.2" rpy="0 0 0"/>
+  <origin xyz="0.002 0.0 0.2" rpy="0 0 0"/>
   <parent link="link__1__1"/>
   <child link="r_a__1__1"/>
@@ -172,5 +172,5 @@
 </joint>
 <joint name="Revolute_5" type="revolute">
-  <origin xyz="0.0505 0.0 0.04" rpy="0 0 0"/>
+  <origin xyz="0.0505 0.0 0.042" rpy="0 0 0"/>
   <parent link="r_a__1__1"/>
   <child link="r_a__2__1"/>
@@ -179,5 +179,5 @@
 </joint>
 <joint name="Revolute_6" type="revolute">
-  <origin xyz="-0.04 0.0 0.0505" rpy="0 0 0"/>
+  <origin xyz="-0.042 0.0 0.0505" rpy="0 0 0"/>
   <parent link="r_a__2__1"/>
   <child link="housing_1"/>

Commit message: Robot model: links 2-3 and 3-4 wear the engraved covers (user parts, text on the outside)
The outer half-shell of each arm link is replaced by the user's cover (부품.stl on link_1, 링크껍데기 (1)_세로.stl
on link__1__1): the old cover faces are removed from the link mesh (faces on the new cover's surface, 6767 / 6769
triangles), the new cover is placed in the link's assembly frame (proper rotations only, text not mirrored; fit
median 0.33 mm, y = the model's 2.984 mm offset) and the engraving faces (floors and walls) are a separate mesh
drawn black.

- orientation chosen by the user: link_1 reads "i - ROBOT" from joint 2 to joint 3 (as on the real arm),
  link__1__1 has "KHU" at the joint 3 end
- meshes/link_1_engraved.stl, link__1__1_engraved.stl (visual + collision), *_engraving.stl (black, visual only);
  the old link meshes stay, unused
- urdf/6dof.urdf, 6dof.xacro, materials.xacro (black), mujoco/6dof_mj.urdf, 6dof.xml, 6dof_control.xml;
  regenerated 6dof_gripper.{urdf,xacro} and pinch_scene.xml (scene sha acd273a728ae)
- inertia unchanged (the covers have the old covers' shape)
- the arm program's model copy is still the old scene, so --real-arm refuses until it is updated

Co-Authored-By: Claude Opus 5.5 <noreply@anthropic.com>

File: 6dof_description/mujoco/6dof_mj.urdf (robot description, URDF)
Before this commit: robot 6dof, 7 links, 6 joints
Links:
- link link_1: geometry collision mesh filename=link_1_engraved.stl scale=0.001 0.001 0.001; visual mesh filename=link_1_engraved.stl scale=0.001 0.001 0.001
- link link__1__1: geometry collision mesh filename=link__1__1_engraved.stl scale=0.001 0.001 0.001; visual mesh filename=link__1__1_engraved.stl scale=0.001 0.001 0.001

File: 6dof_description/urdf/6dof.urdf (robot description, URDF)
Before this commit: robot 6dof, 7 links, 6 joints
Links:
- link link_1: geometry collision mesh filename=package://6dof_description/meshes/link_1_engraved.stl scale=0.001 0.001 0.001; visual mesh filename=package://6dof_description/meshes/link_1_engraved.stl scale=0.001 0.001 0.001
- link link__1__1: geometry collision mesh filename=package://6dof_description/meshes/link__1__1_engraved.stl scale=0.001 0.001 0.001; visual mesh filename=package://6dof_description/meshes/link__1__1_engraved.stl scale=0.001 0.001 0.001

File: 6dof_description/urdf/6dof.xacro (robot description, xacro)
@@ -51,12 +51,19 @@
     <origin xyz="-0.04 -0.002984 -0.092054" rpy="0 0 0"/>
     <geometry>
-      <mesh filename="package://6dof_description/meshes/link_1.stl" scale="0.001 0.001 0.001"/>
-    </geometry>
-    <material name="silver"/>
-  </visual>
-  <collision>
+      <mesh filename="package://6dof_description/meshes/link_1_engraved.stl" scale="0.001 0.001 0.001"/>
+    </geometry>
+    <material name="silver"/>
+  </visual>
+  <visual>
     <origin xyz="-0.04 -0.002984 -0.092054" rpy="0 0 0"/>
     <geometry>
-      <mesh filename="package://6dof_description/meshes/link_1.stl" scale="0.001 0.001 0.001"/>
+      <mesh filename="package://6dof_description/meshes/link_1_engraving.stl" scale="0.001 0.001 0.001"/>
+    </geometry>
+    <material name="black"/>
+  </visual>
+  <collision>
+    <origin xyz="-0.04 -0.002984 -0.092054" rpy="0 0 0"/>
+    <geometry>
+      <mesh filename="package://6dof_description/meshes/link_1_engraved.stl" scale="0.001 0.001 0.001"/>
     </geometry>
   </collision>
@@ -71,12 +78,19 @@
     <origin xyz="-0.04 -0.002984 -0.292054" rpy="0 0 0"/>
     <geometry>
-      <mesh filename="package://6dof_description/meshes/link__1__1.stl" scale="0.001 0.001 0.001"/>
-    </geometry>
-    <material name="silver"/>
-  </visual>
-  <collision>
+      <mesh filename="package://6dof_description/meshes/link__1__1_engraved.stl" scale="0.001 0.001 0.001"/>
+    </geometry>
+    <material name="silver"/>
+  </visual>
+  <visual>
     <origin xyz="-0.04 -0.002984 -0.292054" rpy="0 0 0"/>
     <geometry>
-      <mesh filename="package://6dof_description/meshes/link__1__1.stl" scale="0.001 0.001 0.001"/>
+      <mesh filename="package://6dof_description/meshes/link__1__1_engraving.stl" scale="0.001 0.001 0.001"/>
+    </geometry>
+    <material name="black"/>
+  </visual>
+  <collision>
+    <origin xyz="-0.04 -0.002984 -0.292054" rpy="0 0 0"/>
+    <geometry>
+      <mesh filename="package://6dof_description/meshes/link__1__1_engraved.stl" scale="0.001 0.001 0.001"/>
     </geometry>
   </collision>

File: 6dof_description/urdf/6dof_gripper.urdf (robot description, URDF)
Before this commit: robot 6dof_gripper, 7 links, 6 joints
Links:
- link link_1: geometry collision mesh filename=package://6dof_description/meshes/link_1_engraved.stl scale=0.001 0.001 0.001; visual mesh filename=package://6dof_description/meshes/link_1_engraved.stl scale=0.001 0.001 0.001
- link link__1__1: geometry collision mesh filename=package://6dof_description/meshes/link__1__1_engraved.stl scale=0.001 0.001 0.001; visual mesh filename=package://6dof_description/meshes/link__1__1_engraved.stl scale=0.001 0.001 0.001

File: 6dof_description/urdf/6dof_gripper.xacro (robot description, xacro)
@@ -51,12 +51,19 @@
     <origin xyz="-0.04 -0.002984 -0.092054" rpy="0 0 0"/>
     <geometry>
-      <mesh filename="package://6dof_description/meshes/link_1.stl" scale="0.001 0.001 0.001"/>
-    </geometry>
-    <material name="silver"/>
-  </visual>
-  <collision>
+      <mesh filename="package://6dof_description/meshes/link_1_engraved.stl" scale="0.001 0.001 0.001"/>
+    </geometry>
+    <material name="silver"/>
+  </visual>
+  <visual>
     <origin xyz="-0.04 -0.002984 -0.092054" rpy="0 0 0"/>
     <geometry>
-      <mesh filename="package://6dof_description/meshes/link_1.stl" scale="0.001 0.001 0.001"/>
+      <mesh filename="package://6dof_description/meshes/link_1_engraving.stl" scale="0.001 0.001 0.001"/>
+    </geometry>
+    <material name="black"/>
+  </visual>
+  <collision>
+    <origin xyz="-0.04 -0.002984 -0.092054" rpy="0 0 0"/>
+    <geometry>
+      <mesh filename="package://6dof_description/meshes/link_1_engraved.stl" scale="0.001 0.001 0.001"/>
     </geometry>
   </collision>
@@ -71,12 +78,19 @@
     <origin xyz="-0.04 -0.002984 -0.292054" rpy="0 0 0"/>
     <geometry>
-      <mesh filename="package://6dof_description/meshes/link__1__1.stl" scale="0.001 0.001 0.001"/>
-    </geometry>
-    <material name="silver"/>
-  </visual>
-  <collision>
+      <mesh filename="package://6dof_description/meshes/link__1__1_engraved.stl" scale="0.001 0.001 0.001"/>
+    </geometry>
+    <material name="silver"/>
+  </visual>
+  <visual>
     <origin xyz="-0.04 -0.002984 -0.292054" rpy="0 0 0"/>
     <geometry>
-      <mesh filename="package://6dof_description/meshes/link__1__1.stl" scale="0.001 0.001 0.001"/>
+      <mesh filename="package://6dof_description/meshes/link__1__1_engraving.stl" scale="0.001 0.001 0.001"/>
+    </geometry>
+    <material name="black"/>
+  </visual>
+  <collision>
+    <origin xyz="-0.04 -0.002984 -0.292054" rpy="0 0 0"/>
+    <geometry>
+      <mesh filename="package://6dof_description/meshes/link__1__1_engraved.stl" scale="0.001 0.001 0.001"/>
     </geometry>
   </collision>

File: 6dof_description/urdf/materials.xacro (robot description, xacro)
@@ -4,3 +4,6 @@
   <color rgba="0.700 0.700 0.700 1.000"/>
 </material>
+<material name="black">
+  <color rgba="0.020 0.020 0.020 1.000"/>
+</material>
 </robot>

Commit message: Robot model: orange rings (ID 70 / OD 80 / 6 mm) at link_1's joint 2 end and link__1__1's joint 3 end
Each ring sits on the Ø80 joint housing against the joint face (link_1 x 40-46 mm, link__1__1 x 34-40 mm in the
mesh frame). The ring volume is cut from the link mesh: the end-face rim moves in to r 35, the housing facets start
at the step, and the seat floor (r 35) and step are new faces; open edges are unchanged (517 / 603, from the cover
replacement). The ring is a closed 77-gon on the housing's own rim vertices, so its outside continues the housing.

- meshes/link_1_engraved.stl, link__1__1_engraved.stl (seat cut), new meshes/*_ring.stl (visual, orange
  1.0 0.42 0.0, and collision: the hull of cut link + ring covers the old link hull)
- urdf/6dof.urdf, 6dof.xacro, materials.xacro (orange), mujoco/6dof_mj.urdf, 6dof.xml, 6dof_control.xml;
  regenerated 6dof_gripper.{urdf,xacro} and pinch_scene.xml (scene sha d0885d55d921)
- collision.py: floor_by_body keeps the minimum when a body has several collision geoms
- inertia unchanged
- the arm program's model copy is still 7f96b2c, so --real-arm refuses until it is updated

Co-Authored-By: Claude Opus 5.5 <noreply@anthropic.com>

File: 6dof_description/mujoco/6dof_mj.urdf (robot description, URDF)
Before this commit: robot 6dof, 7 links, 6 joints
Links:
- link link_1: geometry collision mesh filename=link_1_engraved.stl scale=0.001 0.001 0.001; collision mesh filename=link_1_ring.stl scale=0.001 0.001 0.001
- link link__1__1: geometry collision mesh filename=link__1__1_engraved.stl scale=0.001 0.001 0.001; collision mesh filename=link__1__1_ring.stl scale=0.001 0.001 0.001

File: 6dof_description/urdf/6dof.urdf (robot description, URDF)
Before this commit: robot 6dof, 7 links, 6 joints
Links:
- link link_1: geometry collision mesh filename=package://6dof_description/meshes/link_1_engraved.stl scale=0.001 0.001 0.001; collision mesh filename=package://6dof_description/meshes/link_1_ring.stl scale=0.001 0.001 0.001
- link link__1__1: geometry collision mesh filename=package://6dof_description/meshes/link__1__1_engraved.stl scale=0.001 0.001 0.001; collision mesh filename=package://6dof_description/meshes/link__1__1_ring.stl scale=0.001 0.001 0.001

File: 6dof_description/urdf/6dof.xacro (robot description, xacro)
@@ -62,8 +62,21 @@
     <material name="black"/>
   </visual>
+  <visual>
+    <origin xyz="-0.04 -0.002984 -0.092054" rpy="0 0 0"/>
+    <geometry>
+      <mesh filename="package://6dof_description/meshes/link_1_ring.stl" scale="0.001 0.001 0.001"/>
+    </geometry>
+    <material name="orange"/>
+  </visual>
   <collision>
     <origin xyz="-0.04 -0.002984 -0.092054" rpy="0 0 0"/>
     <geometry>
       <mesh filename="package://6dof_description/meshes/link_1_engraved.stl" scale="0.001 0.001 0.001"/>
+    </geometry>
+  </collision>
+  <collision>
+    <origin xyz="-0.04 -0.002984 -0.092054" rpy="0 0 0"/>
+    <geometry>
+      <mesh filename="package://6dof_description/meshes/link_1_ring.stl" scale="0.001 0.001 0.001"/>
     </geometry>
   </collision>
@@ -89,8 +102,21 @@
     <material name="black"/>
   </visual>
+  <visual>
+    <origin xyz="-0.04 -0.002984 -0.292054" rpy="0 0 0"/>
+    <geometry>
+      <mesh filename="package://6dof_description/meshes/link__1__1_ring.stl" scale="0.001 0.001 0.001"/>
+    </geometry>
+    <material name="orange"/>
+  </visual>
   <collision>
     <origin xyz="-0.04 -0.002984 -0.292054" rpy="0 0 0"/>
     <geometry>
       <mesh filename="package://6dof_description/meshes/link__1__1_engraved.stl" scale="0.001 0.001 0.001"/>
+    </geometry>
+  </collision>
+  <collision>
+    <origin xyz="-0.04 -0.002984 -0.292054" rpy="0 0 0"/>
+    <geometry>
+      <mesh filename="package://6dof_description/meshes/link__1__1_ring.stl" scale="0.001 0.001 0.001"/>
     </geometry>
   </collision>

File: 6dof_description/urdf/6dof_gripper.urdf (robot description, URDF)
Before this commit: robot 6dof_gripper, 7 links, 6 joints
Links:
- link link_1: geometry collision mesh filename=package://6dof_description/meshes/link_1_engraved.stl scale=0.001 0.001 0.001; collision mesh filename=package://6dof_description/meshes/link_1_ring.stl scale=0.001 0.001 0.001
- link link__1__1: geometry collision mesh filename=package://6dof_description/meshes/link__1__1_engraved.stl scale=0.001 0.001 0.001; collision mesh filename=package://6dof_description/meshes/link__1__1_ring.stl scale=0.001 0.001 0.001

File: 6dof_description/urdf/6dof_gripper.xacro (robot description, xacro)
@@ -62,8 +62,21 @@
     <material name="black"/>
   </visual>
+  <visual>
+    <origin xyz="-0.04 -0.002984 -0.092054" rpy="0 0 0"/>
+    <geometry>
+      <mesh filename="package://6dof_description/meshes/link_1_ring.stl" scale="0.001 0.001 0.001"/>
+    </geometry>
+    <material name="orange"/>
+  </visual>
   <collision>
     <origin xyz="-0.04 -0.002984 -0.092054" rpy="0 0 0"/>
     <geometry>
       <mesh filename="package://6dof_description/meshes/link_1_engraved.stl" scale="0.001 0.001 0.001"/>
+    </geometry>
+  </collision>
+  <collision>
+    <origin xyz="-0.04 -0.002984 -0.092054" rpy="0 0 0"/>
+    <geometry>
+      <mesh filename="package://6dof_description/meshes/link_1_ring.stl" scale="0.001 0.001 0.001"/>
     </geometry>
   </collision>
@@ -89,8 +102,21 @@
     <material name="black"/>
   </visual>
+  <visual>
+    <origin xyz="-0.04 -0.002984 -0.292054" rpy="0 0 0"/>
+    <geometry>
+      <mesh filename="package://6dof_description/meshes/link__1__1_ring.stl" scale="0.001 0.001 0.001"/>
+    </geometry>
+    <material name="orange"/>
+  </visual>
   <collision>
     <origin xyz="-0.04 -0.002984 -0.292054" rpy="0 0 0"/>
     <geometry>
       <mesh filename="package://6dof_description/meshes/link__1__1_engraved.stl" scale="0.001 0.001 0.001"/>
+    </geometry>
+  </collision>
+  <collision>
+    <origin xyz="-0.04 -0.002984 -0.292054" rpy="0 0 0"/>
+    <geometry>
+      <mesh filename="package://6dof_description/meshes/link__1__1_ring.stl" scale="0.001 0.001 0.001"/>
     </geometry>
   </collision>

File: 6dof_description/urdf/materials.xacro (robot description, xacro)
@@ -7,3 +7,6 @@
   <color rgba="0.020 0.020 0.020 1.000"/>
 </material>
+<material name="orange">
+  <color rgba="1.000 0.420 0.000 1.000"/>
+</material>
 </robot>
