Commit message: Gripper: fingers drawn black
gripper.stl is split into its connected components, triangles unchanged: meshes/gripper_body.stl (mount plate +
housing) and meshes/gripper_fingers.stl (the two tip prongs, 3060 triangles). They are two visual geoms
(gripper_visual grey, gripper_fingers_visual black 0.02); the collision geom stays the whole gripper.stl (mass,
inertia, hull unchanged) and moves to group 3 (hidden), otherwise its grey would be drawn over the fingers.

- configs/demo.json gripper: body_mesh, fingers_mesh, fingers_rgba (+ note)
- gripper.py: visual_parts(); the URDF/xacro variants get a second <visual> (material black)
- regenerated 6dof_gripper.{urdf,xacro} and pinch_scene.xml
- test_gripper: split = gripper.stl, colours, groups

Co-Authored-By: Claude Opus 5.5 <noreply@anthropic.com>

File: 6dof_description/urdf/6dof_gripper.urdf (robot description, URDF)
Before this commit: robot 6dof_gripper, 7 links, 6 joints
Links:
- link housing_1: geometry collision mesh filename=package://6dof_description/meshes/gripper.stl scale=0.001 0.001 0.001; visual mesh filename=package://6dof_description/meshes/gripper_body.stl scale=0.001 0.001 0.001

File: 6dof_description/urdf/6dof_gripper.xacro (robot description, xacro)
@@ -172,7 +172,14 @@
     <origin xyz="0.063911 0.242590 0.114841" rpy="-1.570796 -0.000000 1.570796"/>
     <geometry>
-      <mesh filename="package://6dof_description/meshes/gripper.stl" scale="0.001 0.001 0.001"/>
-    </geometry>
-    <material name="silver"/>
+      <mesh filename="package://6dof_description/meshes/gripper_body.stl" scale="0.001 0.001 0.001"/>
+    </geometry>
+    <material name="silver"/>
+  </visual>
+  <visual>
+    <origin xyz="0.063911 0.242590 0.114841" rpy="-1.570796 -0.000000 1.570796"/>
+    <geometry>
+      <mesh filename="package://6dof_description/meshes/gripper_fingers.stl" scale="0.001 0.001 0.001"/>
+    </geometry>
+    <material name="black"/>
   </visual>
   <collision>
